Commit message: finished week2

File: src/hrwros_week2/urdf/hrwros_assignment1.xacro (robot description, xacro)
@@ -72,3 +72,10 @@
   </joint>
   <!-- Add your solution to assignment 1 here -->
+  <xacro:bin_urdf prefix="bin_2_"/>
+  <!-- bin 2 -->
+  <joint name="bin_2_joint" type="fixed">
+    <parent link="world_interface" />
+	<child link="bin_2_base_link" />
+	<origin xyz="2.5 1.84 0" rpy="0 0 0" />
+  </joint>
 </robot>

File: src/hrwros_week2/urdf/hrwros_assignment2.xacro (robot description, xacro)
@@ -72,3 +72,19 @@
   </joint>
   <!-- Add your solution to assignment 2 here -->
+  <link name="sphere_link">
+    <visual>
+	<origin xyz="0 0 0" />
+	<geometry>
+	  <sphere radius="0.4"/>
+	</geometry>
+	<material name="green">
+	   <color rgba="0 1 0 1"/>
+	</material>
+    </visual>
+   </link>
+   <joint name="sphere_joint" type="fixed">
+     <origin xyz="5.8 -5.21 0.4"/>
+     <parent link="world"/>
+     <child link="sphere_link"/>
+   </joint>
 </robot>
